File: pcb-files/implant/mmimplant.brd (EAGLE design)
At the start: 27.3 x 19.1 mm, 15 parts, among them IC2 ATMEGA32U4-MU

Commit message: Workin on the implant
Parts:
- added IC1: TPS7A2650DRVR, SamacSys_Parts:SON65P200X200X80-7N
Connections:
- removed net VCC: 5V.TP, IC2.14
- new net 5V: IC1.1, IC2.2
- net GND: now also IC1.3, IC1.5, IC1.7
- net VCC1: now also IC2.14
- net VIN: now also 5V.TP, IC1.4, IC1.6; no longer IC2.2
Routing:
- net VIN: track 8.23 -> 27.7 mm
Changed lines of the file:
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@@
 <attribute name="VALUE" x="20.32" y="0" size="1.27" layer="27"/>
+</element>
+<element name="IC1" library="SamacSys_Parts" package="SON65P200X200X80-7N" value="TPS7A2650DRVR" x="20.0025" y="12.7" smashed="yes" rot="MR90">
+<attribute name="DESCRIPTION" value="LDO Voltage Regulators 500-mA 18-V ultra-low-IQ low-dropout (LDO) linear voltage regulator with power good 6-WSON -40 to 125" x="20.0025" y="12.7" size="1.778" layer="28" rot="MR90" display="off"/>
+<attribute name="HEIGHT" value="0.8mm" x="20.0025" y="12.7" size="1.778" layer="28" rot="MR90" display="off"/>
+<attribute name="MANUFACTURER_NAME" value="Texas Instruments" x="20.0025" y="12.7" size="1.778" layer="28" rot="MR90" display="off"/>
+<attribute name="MANUFACTURER_PART_NUMBER" value="TPS7A2650DRVR" x="20.0025" y="12.7" size="1.778" layer="28" rot="MR90" display="off"/>
+<attribute name="MOUSER_PART_NUMBER" value="595-TPS7A2650DRVR" x="20.0025" y="12.7" size="1.778" layer="28" rot="MR90" display="off"/>
+<attribute name="MOUSER_PRICE-STOCK" value="https://www.mouser.co.uk/ProductDetail/Texas-Instruments/TPS7A2650DRVR?qs=OTrKUuiFdkaeaXj%2F%252BB59oA%3D%3D" x="20.0025" y="12.7" size="1.778" layer="28" rot="MR90" display="off"/>
 </element>
 </elements>
@@
 <contactref element="JP2" pad="4"/>
 <contactref element="JP1" pad="1"/>
+<contactref element="IC1" pad="5"/>
+<contactref element="IC1" pad="3"/>
+<contactref element="IC1" pad="7"/>
 </signal>
 <signal name="CAPS">
@@
 <wire x1="9.71323125" y1="6.5414" x2="15.1139" y2="6.5414" width="0.1524" layer="16"/>
 <wire x1="15.1139" y1="6.5414" x2="16.51" y2="7.9375" width="0.1524" layer="16"/>
-</signal>
-<signal name="VIN">
-<contactref element="USB-C" pad="A4"/>
-<contactref element="USB-C" pad="B9"/>
-<contactref element="USB-C" pad="A9"/>
-<contactref element="USB-C" pad="B4"/>
-<contactref element="IC2" pad="2"/>
-<wire x1="11.21" y1="12.8025" x2="11.21" y2="14.1525" width="0.2032" layer="1"/>
-<wire x1="15.46" y1="12.8025" x2="15.46" y2="14.1525" width="0.2032" layer="1"/>
-<wire x1="11.21" y1="14.1525" x2="11.21" y2="14.7025" width="0.1524" layer="16"/>
-<wire x1="11.21" y1="14.7025" x2="11.43" y2="14.9225" width="0.1524" layer="16"/>
-<wire x1="15.24" y1="14.9225" x2="15.46" y2="14.7025" width="0.1524" layer="16"/>
-<wire x1="15.46" y1="14.7025" x2="15.46" y2="14.1525" width="0.1524" layer="16"/>
-<wire x1="11.43" y1="14.9225" x2="15.24" y2="14.9225" width="0.1524" layer="16"/>
-<wire x1="15.46" y1="12.8025" x2="15.335" y2="9.4325" width="0" layer="19" extent="1-1"/>
 </signal>
 <signal name="CC">
@@
 <contactref element="IC2" pad="4"/>
 <wire x1="18.5728125" y1="8.1589" x2="18.1214" y2="8.6103125" width="0.1524" layer="1"/>
-<wire x1="18.1214" y1="8.6103125" x2="18.1214" y2="8.8661" width="0.1524" layer="1"/>
-<wire x1="18.1214" y1="8.8661" x2="16.51" y2="10.4775" width="0.1524" layer="1"/>
+<wire x1="18.1214" y1="8.6103125" x2="18.1214" y2="9.5011" width="0.1524" layer="1"/>
+<wire x1="18.1214" y1="9.5011" x2="17.145" y2="10.4775" width="0.1524" layer="1"/>
 <wire x1="21.2725" y1="7.255" x2="20.6232875" y2="7.255" width="0.1524" layer="1"/>
 <wire x1="20.6232875" y1="7.255" x2="19.7193875" y2="8.1589" width="0.1524" layer="1"/>
 <wire x1="19.7193875" y1="8.1589" x2="18.5728125" y2="8.1589" width="0.1524" layer="1"/>
-<wire x1="16.51" y1="10.4775" x2="14.605" y2="10.4775" width="0.1524" layer="1"/>
+<wire x1="17.145" y1="10.4775" x2="14.605" y2="10.4775" width="0.1524" layer="1"/>
 <wire x1="14.605" y1="10.4775" x2="14.2875" y2="10.16" width="0.1524" layer="1"/>
 <wire x1="14.2875" y1="10.16" x2="14.2875" y2="9.48" width="0.1524" layer="1"/>
@@
 <contactref element="R3" pad="2"/>
 <contactref element="IC2" pad="3"/>
-<wire x1="14.9225" y1="10.16" x2="16.145" y2="10.16" width="0.1524" layer="1"/>
+<wire x1="14.9225" y1="10.16" x2="16.78" y2="10.16" width="0.1524" layer="1"/>
 <wire x1="14.9225" y1="10.16" x2="14.835" y2="10.0725" width="0.1524" layer="1"/>
 <wire x1="14.835" y1="10.0725" x2="14.835" y2="9.4325" width="0.1524" layer="1"/>
-<wire x1="16.145" y1="10.16" x2="17.78" y2="8.525" width="0.1524" layer="1"/>
-<wire x1="17.78" y1="8.525" x2="17.78" y2="7.9375" width="0.1524" layer="1"/>
+<wire x1="16.78" y1="10.16" x2="17.78" y2="9.16" width="0.1524" layer="1"/>
+<wire x1="17.78" y1="9.16" x2="17.78" y2="7.9375" width="0.1524" layer="1"/>
 <wire x1="17.78" y1="7.9375" x2="18.4625" y2="7.255" width="0.1524" layer="1"/>
 <wire x1="18.4625" y1="7.255" x2="19.05" y2="7.255" width="0.1524" layer="1"/>
@@
 <contactref element="RST" pad="TP"/>
 <wire x1="9.935" y1="8.0325" x2="13.335" y2="5.08" width="0" layer="19" extent="1-16"/>
-</signal>
-<signal name="VCC">
-<contactref element="IC2" pad="14"/>
-<contactref element="5V" pad="TP"/>
-<wire x1="9.935" y1="7.5325" x2="16.51" y2="5.08" width="0" layer="19" extent="1-16"/>
 </signal>
 <signal name="SCROLL">
@@
 <wire x1="11.43" y1="2.5375" x2="11.335" y2="2.6325" width="0.2032" layer="1"/>
 <wire x1="6.6675" y1="1.5875" x2="11.1125" y2="1.5875" width="0.2032" layer="1"/>
+<contactref element="IC2" pad="14"/>
+<wire x1="11.335" y1="2.6325" x2="9.935" y2="7.5325" width="0" layer="19" extent="1-1"/>
 </signal>
 <signal name="DATA">
@@
 <contactref element="JP2" pad="5"/>
 </signal>
+<signal name="VIN">
+<contactref element="IC1" pad="4"/>
+<contactref element="IC1" pad="6"/>
+<contactref element="USB-C" pad="A4"/>
+<contactref element="USB-C" pad="B9"/>
+<contactref element="USB-C" pad="A9"/>
+<contactref element="USB-C" pad="B4"/>
+<wire x1="11.21" y1="12.8025" x2="11.21" y2="14.1525" width="0.2032" layer="1"/>
+<wire x1="15.46" y1="12.8025" x2="15.46" y2="14.1525" width="0.2032" layer="1"/>
+<wire x1="11.21" y1="14.1525" x2="11.21" y2="14.7025" width="0.1524" layer="16"/>
+<wire x1="11.21" y1="14.7025" x2="11.43" y2="14.9225" width="0.1524" layer="16"/>
+<wire x1="15.24" y1="14.9225" x2="15.46" y2="14.7025" width="0.1524" layer="16"/>
+<wire x1="15.46" y1="14.7025" x2="15.46" y2="14.1525" width="0.1524" layer="16"/>
+<wire x1="11.43" y1="14.9225" x2="15.24" y2="14.9225" width="0.1524" layer="16"/>
+<wire x1="15.46" y1="14.1525" x2="16.5475" y2="15.24" width="0.2032" layer="16"/>
+<wire x1="18.7325" y1="15.24" x2="19.05" y2="14.9225" width="0.2032" layer="16"/>
+<wire x1="19.05" y1="14.9225" x2="19.3675" y2="14.605" width="0.2032" layer="16"/>
+<wire x1="19.3675" y1="14.605" x2="19.3675" y2="13.765" width="0.2032" layer="16"/>
+<wire x1="19.3675" y1="13.765" x2="19.3525" y2="13.75" width="0.2032" layer="16"/>
+<wire x1="16.5475" y1="15.24" x2="18.7325" y2="15.24" width="0.2032" layer="16"/>
+<wire x1="20.6525" y1="13.75" x2="20.6375" y2="13.765" width="0.2032" layer="16"/>
+<wire x1="20.6375" y1="14.605" x2="20.6375" y2="13.765" width="0.2032" layer="16"/>
+<wire x1="20.32" y1="14.9225" x2="19.05" y2="14.9225" width="0.2032" layer="16"/>
+<wire x1="20.32" y1="14.9225" x2="20.6375" y2="14.605" width="0.2032" layer="16"/>
+<wire x1="19.05" y1="14.9225" x2="18.415" y2="14.2875" width="0.2032" layer="16"/>
+<wire x1="18.415" y1="14.2875" x2="18.415" y2="6.0325" width="0.2032" layer="16"/>
+<contactref element="5V" pad="TP"/>
+<wire x1="17.4625" y1="5.08" x2="16.51" y2="5.08" width="0.2032" layer="16"/>
+<wire x1="18.415" y1="6.0325" x2="17.4625" y2="5.08" width="0.2032" layer="16"/>
+</signal>
+<signal name="5V">
+<contactref element="IC1" pad="1"/>
+<contactref element="IC2" pad="2"/>
+<wire x1="15.335" y1="9.4325" x2="20.6525" y2="11.65" width="0" layer="19" extent="1-16"/>
+</signal>
 </signals>

Commit message: Finishing touches on implant + gerber
Parts:
- moved C1 0.63 mm to (6.99, 12.1)
- moved R1 0.45 mm to (6.99, 15.9)
Routing:
- net RST: track 0.00 -> 8.58 mm, vias 0 -> 1
- net 5V: track 0.00 -> 7.28 mm, vias 0 -> 1
- net SCLK: track 17.0 -> 22.9 mm
- net MOSI: track 11.7 -> 13.5 mm
- net VCC1: track 8.35 -> 10.1 mm, vias 0 -> 1
- net VIN: track 27.7 -> 29.4 mm
- net D+RES: track 9.72 -> 11.0 mm
- net D-RES: track 6.81 -> 8.08 mm
- net D-: track 9.31 -> 10.2 mm
- net D+: track 10.7 -> 11.4 mm
