File: pcb-files/implant/mmimplant.sch (EAGLE design)
At the start: 15 parts, among them IC2 ATMEGA32U4-MU

Commit message: Workin on the implant
Parts:
- added IC1: TPS7A2650DRVR, SamacSys_Parts:TPS7A2650DRVR
Connections:
- removed net VCC: 5V.TP, IC2.VCC_1
- new net 5V: IC1.OUT, IC2.UVCC
- net GND: now also IC1.EP, IC1.GND, IC1.PG
- net VCC1: now also IC2.VCC_1
- net VIN: now also 5V.TP, IC1.EN, IC1.IN; no longer IC2.UVCC
Changed lines of the file:
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@@
 <part name="GND9" library="supply1" library_urn="urn:adsk.eagle:library:371" deviceset="GND" device=""/>
 <part name="JP1" library="pinhead" library_urn="urn:adsk.eagle:library:325" deviceset="PINHD-1X1" device="" package3d_urn="urn:adsk.eagle:package:22485/2"/>
+<part name="IC1" library="SamacSys_Parts" deviceset="TPS7A2650DRVR" device=""/>
+<part name="GND1" library="supply1" library_urn="urn:adsk.eagle:library:371" deviceset="GND" device=""/>
 </parts>
 <sheets>
@@
 <attribute name="TP_SIGNAL_NAME" x="100.33" y="-3.81" size="1.778" layer="97" rot="R180"/>
 </instance>
-<instance part="5V" gate="G$1" x="104.14" y="-5.08" smashed="yes" rot="R180">
-<attribute name="TP_SIGNAL_NAME" x="102.87" y="-3.81" size="1.778" layer="97" rot="R180"/>
+<instance part="5V" gate="G$1" x="60.96" y="88.9" smashed="yes" rot="R270">
+<attribute name="TP_SIGNAL_NAME" x="59.69" y="87.63" size="1.778" layer="97" rot="R270"/>
 </instance>
 <instance part="GND" gate="G$1" x="106.68" y="-5.08" smashed="yes" rot="R180">
@@
 <instance part="JP1" gate="G$1" x="124.46" y="114.3" smashed="yes" rot="R90">
 <attribute name="VALUE" x="129.54" y="107.95" size="1.778" layer="96" rot="R90"/>
+</instance>
+<instance part="IC1" gate="G$1" x="25.4" y="88.9" smashed="yes">
+<attribute name="NAME" x="46.99" y="96.52" size="1.778" layer="95" align="center-left"/>
+<attribute name="VALUE" x="46.99" y="93.98" size="1.778" layer="96" align="center-left"/>
+</instance>
+<instance part="GND1" gate="1" x="53.34" y="86.36" smashed="yes" rot="R90">
+<attribute name="VALUE" x="55.88" y="83.82" size="1.778" layer="96" rot="R90"/>
 </instance>
 </instances>
@@
 <pinref part="GND" gate="G$1" pin="TP"/>
 <pinref part="IC2" gate="G$1" pin="GND_1"/>
-<pinref part="IC2" gate="G$1" pin="GND_1"/>
 <junction x="106.68" y="-2.54"/>
 <junction x="106.68" y="-2.54"/>
@@
 <pinref part="JP2" gate="A" pin="4"/>
 <pinref part="GND9" gate="1" pin="GND"/>
+</segment>
+<segment>
+<pinref part="GND1" gate="1" pin="GND"/>
+<pinref part="IC1" gate="G$1" pin="GND"/>
+<wire x1="50.8" y1="86.36" x2="55.88" y2="86.36" width="0.1524" layer="91"/>
+<junction x="50.8" y="86.36"/>
+<pinref part="IC1" gate="G$1" pin="PG"/>
+<wire x1="25.4" y1="83.82" x2="25.4" y2="81.28" width="0.1524" layer="91"/>
+<wire x1="55.88" y1="81.28" x2="50.8" y2="81.28" width="0.1524" layer="91"/>
+<wire x1="50.8" y1="81.28" x2="25.4" y2="81.28" width="0.1524" layer="91"/>
+<wire x1="55.88" y1="81.28" x2="55.88" y2="86.36" width="0.1524" layer="91"/>
+<pinref part="IC1" gate="G$1" pin="EP"/>
+<wire x1="38.1" y1="71.12" x2="50.8" y2="71.12" width="0.1524" layer="91"/>
+<wire x1="50.8" y1="71.12" x2="50.8" y2="81.28" width="0.1524" layer="91"/>
+<junction x="50.8" y="81.28"/>
 </segment>
 </net>
@@
 <pinref part="SCLK" gate="G$1" pin="TP"/>
 <pinref part="IC2" gate="G$1" pin="(PCINT1/SCLK)_PB1"/>
-</segment>
-</net>
-<net name="VIN" class="0">
-<segment>
-<wire x1="43.18" y1="66.04" x2="43.18" y2="33.02" width="0.1524" layer="91"/>
-<wire x1="43.18" y1="33.02" x2="10.16" y2="33.02" width="0.1524" layer="91"/>
-<pinref part="USB-C" gate="G$1" pin="VBUS"/>
-<wire x1="43.18" y1="66.04" x2="71.12" y2="66.04" width="0.1524" layer="91"/>
-<pinref part="IC2" gate="G$1" pin="UVCC"/>
 </segment>
 </net>
@@
 <pinref part="IC2" gate="G$1" pin="!RESET"/>
 <pinref part="RST" gate="G$1" pin="TP"/>
-</segment>
-</net>
-<net name="VCC" class="0">
-<segment>
-<pinref part="IC2" gate="G$1" pin="VCC_1"/>
-<pinref part="5V" gate="G$1" pin="TP"/>
 </segment>
 </net>
@@
 <wire x1="167.64" y1="55.88" x2="187.96" y2="55.88" width="0.1524" layer="91"/>
 <wire x1="187.96" y1="55.88" x2="187.96" y2="58.42" width="0.1524" layer="91"/>
+<pinref part="IC2" gate="G$1" pin="VCC_1"/>
 </segment>
 </net>
@@
 </segment>
 </net>
+<net name="VIN" class="0">
+<segment>
+<pinref part="IC1" gate="G$1" pin="EN"/>
+<wire x1="50.8" y1="83.82" x2="58.42" y2="83.82" width="0.1524" layer="91"/>
+<pinref part="IC1" gate="G$1" pin="IN"/>
+<wire x1="58.42" y1="83.82" x2="58.42" y2="88.9" width="0.1524" layer="91"/>
+<wire x1="58.42" y1="88.9" x2="50.8" y2="88.9" width="0.1524" layer="91"/>
+<wire x1="35.56" y1="33.02" x2="10.16" y2="33.02" width="0.1524" layer="91"/>
+<pinref part="USB-C" gate="G$1" pin="VBUS"/>
+<wire x1="35.56" y1="33.02" x2="35.56" y2="68.58" width="0.1524" layer="91"/>
+<wire x1="35.56" y1="68.58" x2="58.42" y2="68.58" width="0.1524" layer="91"/>
+<wire x1="58.42" y1="83.82" x2="58.42" y2="68.58" width="0.1524" layer="91"/>
+<junction x="58.42" y="83.82"/>
+<pinref part="5V" gate="G$1" pin="TP"/>
+<junction x="58.42" y="88.9"/>
+</segment>
+</net>
+<net name="5V" class="0">
+<segment>
+<pinref part="IC1" gate="G$1" pin="OUT"/>
+<wire x1="25.4" y1="88.9" x2="22.86" y2="88.9" width="0.1524" layer="91"/>
+<wire x1="22.86" y1="88.9" x2="22.86" y2="66.04" width="0.1524" layer="91"/>
+<pinref part="IC2" gate="G$1" pin="UVCC"/>
+<wire x1="22.86" y1="66.04" x2="71.12" y2="66.04" width="0.1524" layer="91"/>
+</segment>
+</net>
