File: pcb-files/keypad/keypad.brd (EAGLE design)
At the start: 61 x 52.1 mm, 23 parts, among them IC2 ATMEGA32U4-MU, J2 SS-60300-046, SW1 CHERRY-MX, SW2 CHERRY-MX, SW3 CHERRY-MX, SW4 CHERRY-MX, SW5 CHERRY-MX, SW6 CHERRY-MX

Commit message: Finished the last board design
Parts:
- moved R2 0.16 mm to (74.3, 75.1)
Routing:
- net VCC: track 12.5 -> 49.5 mm
- net CAPS: track 0.00 -> 25.6 mm, vias 0 -> 1
- net SCRL: track 0.00 -> 18.4 mm, vias 0 -> 1
- net NUM: track 0.00 -> 14.6 mm, vias 0 -> 1
- net GND: track 0.00 -> 1.96 mm, vias 0 -> 4
Changed lines of the file:
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@@
 <attribute name="NAME" x="70.83425" y="77.56525" size="0.8128" layer="26" font="vector" rot="MR180"/>
 </element>
-<element name="R2" library="adafruit" package="R0805" value="22Ω" x="74.295" y="75.2475" smashed="yes" rot="MR0">
-<attribute name="NAME" x="70.83425" y="75.5015" size="0.8128" layer="26" font="vector" rot="MR180"/>
+<element name="R2" library="adafruit" package="R0805" value="22Ω" x="74.295" y="75.08875" smashed="yes" rot="MR0">
+<attribute name="NAME" x="70.83425" y="75.34275" size="0.8128" layer="26" font="vector" rot="MR180"/>
 </element>
 <element name="USB-C" library="USB4085-GF-A_REVA" package="GCT_USB4085-GF-A_REVA" value="USB4085-GF-A_REVA" x="83.66125" y="78.89875" smashed="yes" rot="R180">
@@
 <contactref element="NUM" pad="1"/>
 <contactref element="SCROLL" pad="1"/>
+<via x="71.27875" y="68.8975" extent="1-16" drill="0.35" shape="octagon"/>
+<via x="69.85" y="71.12" extent="1-16" drill="0.35" shape="octagon"/>
+<via x="65.0875" y="70.00875" extent="1-16" drill="0.35" shape="octagon"/>
+<wire x1="65.77" y1="71.68875" x2="65.77" y2="71.1715125" width="0.1524" layer="16"/>
+<wire x1="65.77" y1="71.1715125" x2="65.23355" y2="70.6350625" width="0.1524" layer="16"/>
+<wire x1="65.23355" y1="70.1548" x2="65.0875" y2="70.00875" width="0.1524" layer="16"/>
+<wire x1="65.23355" y1="70.6350625" x2="65.23355" y2="70.1548" width="0.1524" layer="16"/>
+<via x="71.755" y="74.13625" extent="1-16" drill="0.35" shape="octagon"/>
+<wire x1="68.17" y1="75.58875" x2="66.77" y2="78.48875" width="0" layer="19" extent="16-16"/>
 <wire x1="61.37" y1="72.58875" x2="61.11875" y2="70.89625" width="0" layer="19" extent="1-16"/>
+<wire x1="62.77" y1="78.48875" x2="66.77" y2="78.48875" width="0" layer="19" extent="16-16"/>
 </signal>
 <signal name="VIN">
@@
 <wire x1="84.08625" y1="74.87375" x2="84.08625" y2="74.23875" width="0.1524" layer="16"/>
 <wire x1="84.08625" y1="74.23875" x2="83.5075" y2="73.66" width="0.1524" layer="16"/>
-<wire x1="77.7875" y1="73.66" x2="76.2" y2="75.2475" width="0.1524" layer="16"/>
-<wire x1="76.2" y1="75.2475" x2="75.295" y2="75.2475" width="0.1524" layer="16"/>
+<wire x1="77.7875" y1="73.66" x2="76.35875" y2="75.08875" width="0.1524" layer="16"/>
+<wire x1="76.35875" y1="75.08875" x2="75.295" y2="75.08875" width="0.1524" layer="16"/>
 <wire x1="83.5075" y1="73.66" x2="77.7875" y2="73.66" width="0.1524" layer="16"/>
 </signal>
@@
 <contactref element="R2" pad="2"/>
 <contactref element="IC2" pad="4"/>
-<wire x1="73.295" y1="75.2475" x2="72.45375" y2="76.08875" width="0.1524" layer="16"/>
-<wire x1="72.45375" y1="76.08875" x2="68.17" y2="76.08875" width="0.1524" layer="16"/>
+<wire x1="73.295" y1="75.08875" x2="72.295" y2="76.08875" width="0.1524" layer="16"/>
+<wire x1="72.295" y1="76.08875" x2="68.17" y2="76.08875" width="0.1524" layer="16"/>
 </signal>
 <signal name="UCAP">
@@
 <wire x1="51.70875" y1="70.00875" x2="50.57375" y2="71.14375" width="0.2032" layer="16"/>
 <wire x1="57.0120375" y1="70.00875" x2="51.70875" y2="70.00875" width="0.2032" layer="16"/>
-<wire x1="66.27" y1="71.68875" x2="92.86875" y2="56.99125" width="0" layer="19" extent="16-16"/>
+<wire x1="92.86875" y1="56.99125" x2="91.59875" y2="58.26125" width="0.2032" layer="16"/>
+<wire x1="91.59875" y1="58.26125" x2="91.59875" y2="62.5475" width="0.2032" layer="16"/>
+<wire x1="91.59875" y1="62.5475" x2="87.16645" y2="66.9798" width="0.2032" layer="16"/>
+<wire x1="87.16645" y1="66.9798" x2="70.5636875" y2="66.9798" width="0.2032" layer="16"/>
+<wire x1="70.5636875" y1="66.9798" x2="68.0109875" y2="69.5325" width="0.2032" layer="16"/>
+<wire x1="66.04" y1="69.5325" x2="65.88125" y2="69.69125" width="0.2032" layer="16"/>
+<wire x1="66.174" y1="71.1085375" x2="66.174" y2="71.59275" width="0.2032" layer="16"/>
+<wire x1="66.174" y1="71.59275" x2="66.27" y2="71.68875" width="0.2032" layer="16"/>
+<wire x1="65.88125" y1="70.8157875" x2="66.174" y2="71.1085375" width="0.2032" layer="16"/>
+<wire x1="68.0109875" y1="69.5325" x2="66.04" y2="69.5325" width="0.2032" layer="16"/>
+<wire x1="65.88125" y1="69.69125" x2="65.88125" y2="70.8157875" width="0.2032" layer="16"/>
+<wire x1="66.27" y1="71.68875" x2="67.27" y2="78.48875" width="0" layer="19" extent="16-16"/>
 <wire x1="61.37" y1="73.08875" x2="66.27" y2="71.68875" width="0" layer="19" extent="16-16"/>
-<wire x1="67.27" y1="78.48875" x2="66.27" y2="71.68875" width="0" layer="19" extent="16-16"/>
 </signal>
 <signal name="SW1">
@@
 <contactref element="IC2" pad="38"/>
 <contactref element="CAPS" pad="2"/>
-<wire x1="64.92875" y1="72.29625" x2="64.27" y2="78.48875" width="0" layer="19" extent="1-16"/>
+<wire x1="64.27" y1="78.48875" x2="64.3914" y2="78.61015" width="0.1524" layer="16"/>
+<wire x1="64.3914" y1="78.61015" x2="64.3914" y2="79.0584375" width="0.1524" layer="16"/>
+<wire x1="64.3914" y1="79.0584375" x2="64.8667125" y2="79.53375" width="0.1524" layer="16"/>
+<wire x1="70.00875" y1="79.53375" x2="70.8025" y2="78.74" width="0.1524" layer="16"/>
+<wire x1="64.8667125" y1="79.53375" x2="70.00875" y2="79.53375" width="0.1524" layer="16"/>
+<via x="70.8025" y="78.74" extent="1-16" drill="0.35" shape="octagon"/>
+<wire x1="70.8025" y1="78.74" x2="70.8025" y2="70.8025" width="0.1524" layer="1"/>
+<wire x1="70.8025" y1="70.8025" x2="69.37375" y2="69.37375" width="0.1524" layer="1"/>
+<wire x1="64.29375" y1="71.66125" x2="64.29375" y2="69.69125" width="0.1524" layer="1"/>
+<wire x1="64.29375" y1="71.66125" x2="64.92875" y2="72.29625" width="0.1524" layer="1"/>
+<wire x1="64.29375" y1="69.69125" x2="64.61125" y2="69.37375" width="0.1524" layer="1"/>
+<wire x1="64.61125" y1="69.37375" x2="69.37375" y2="69.37375" width="0.1524" layer="1"/>
 </signal>
 <signal name="NUM">
 <contactref element="IC2" pad="37"/>
 <contactref element="NUM" pad="2"/>
-<wire x1="61.11875" y1="72.29625" x2="63.77" y2="78.48875" width="0" layer="19" extent="1-16"/>
+<wire x1="63.77" y1="78.48875" x2="63.6486" y2="78.61015" width="0.1524" layer="16"/>
+<wire x1="63.6486" y1="78.61015" x2="63.6486" y2="79.5346875" width="0.1524" layer="16"/>
+<wire x1="63.6486" y1="79.5346875" x2="63.1732875" y2="80.01" width="0.1524" layer="16"/>
+<wire x1="63.1732875" y1="80.01" x2="60.325" y2="80.01" width="0.1524" layer="16"/>
+<wire x1="60.325" y1="80.01" x2="58.89625" y2="78.58125" width="0.1524" layer="16"/>
+<wire x1="58.89625" y1="78.58125" x2="58.89625" y2="76.35875" width="0.1524" layer="16"/>
+<via x="58.89625" y="76.35875" extent="1-16" drill="0.35" shape="octagon"/>
+<wire x1="58.89625" y1="76.35875" x2="58.89625" y2="73.18375" width="0.1524" layer="1"/>
+<wire x1="59.78375" y1="72.29625" x2="61.11875" y2="72.29625" width="0.1524" layer="1"/>
+<wire x1="58.89625" y1="73.18375" x2="59.78375" y2="72.29625" width="0.1524" layer="1"/>
 </signal>
 <signal name="SCRL">
 <contactref element="IC2" pad="36"/>
 <contactref element="SCROLL" pad="2"/>
-<wire x1="63.27" y1="78.48875" x2="68.73875" y2="72.29625" width="0" layer="19" extent="1-16"/>
+<wire x1="63.30735" y1="79.2171875" x2="63.30735" y2="78.5261" width="0.1524" layer="16"/>
+<wire x1="63.27" y1="78.48875" x2="63.30735" y2="78.5261" width="0.1524" layer="16"/>
+<wire x1="63.30735" y1="79.2171875" x2="62.8320375" y2="79.6925" width="0.1524" layer="16"/>
+<wire x1="60.43855625" y1="79.6925" x2="59.270528125" y2="78.524471875" width="0.1524" layer="16"/>
+<wire x1="62.8320375" y1="79.6925" x2="60.43855625" y2="79.6925" width="0.1524" layer="16"/>
+<wire x1="59.270528125" y1="78.524471875" x2="59.270528125" y2="76.936971875" width="0.1524" layer="16"/>
+<wire x1="59.270528125" y1="76.936971875" x2="59.84875" y2="76.35875" width="0.1524" layer="16"/>
+<via x="59.84875" y="76.35875" extent="1-16" drill="0.35" shape="octagon"/>
+<wire x1="59.84875" y1="76.35875" x2="63.8175" y2="76.35875" width="0.1524" layer="1"/>
+<wire x1="67.88" y1="72.29625" x2="68.73875" y2="72.29625" width="0.1524" layer="1"/>
+<wire x1="63.8175" y1="76.35875" x2="67.88" y2="72.29625" width="0.1524" layer="1"/>
 </signal>
 </signals>
